Commit message: add common macro for sphere and update common macro API

File: xacro4sdf/common.xacro (robot description, xacro)
@@ -25,4 +25,16 @@
         </inertia>
     </xacro_define_macro>
+    <!--macro defination:inertia_sphere-->
+    <xacro_define_macro name="inertia_sphere" params="m r">
+        <mass>${m}</mass>
+        <inertia>
+            <ixx>${2*m*r*r/5}</ixx>
+            <ixy>0</ixy>
+            <ixz>0</ixz>
+            <iyy>${2*m*r*r/5}</iyy>
+            <iyz>0</iyz>
+            <izz>${2*m*r*r/5}</izz>
+        </inertia>
+    </xacro_define_macro>
     <!--macro defination:geometry cylinder-->
     <xacro_define_macro name="geometry_cylinder" params="r l">
@@ -42,18 +54,26 @@
         </geometry>
     </xacro_define_macro>
+    <!--macro defination:geometry sphere-->
+    <xacro_define_macro name="geometry_sphere" params="r">
+        <geometry>
+            <sphere>
+                <radius>${r}</radius>
+            </sphere>
+        </geometry>
+    </xacro_define_macro>
     <!--macro defination:geometry mesh-->
-    <xacro_define_macro name="geometry_mesh" params="filename">
+    <xacro_define_macro name="geometry_mesh" params="uri">
         <geometry>
             <mesh>
-                <uri>${filename}</uri>
+                <uri>${uri}</uri>
             </mesh>
         </geometry>
     </xacro_define_macro>
     <!--macro defination:visual_collision_with_mesh-->
-    <xacro_define_macro name="visual_collision_with_mesh" params="prefix filename">
+    <xacro_define_macro name="visual_collision_with_mesh" params="prefix uri">
         <visual name="${prefix}_visual">
             <geometry>
                 <mesh>
-                    <uri>${filename}</uri>
+                    <uri>${uri}</uri>
                 </mesh>
             </geometry>
@@ -62,5 +82,5 @@
             <geometry>
                 <mesh>
-                    <uri>${filename}</uri>
+                    <uri>${uri}</uri>
                 </mesh>
             </geometry>
