Commit message: add include and update api

File: test/model.sdf.xacro (robot description, xacro)
@@ -1,16 +1,5 @@
 <?xml version="1.0"?>
 <sdf version="1.7">
-    <xacro_property name="h" value="0.2" />
-    <xacro_macro_define macro_name="inertia_box" params="m x y z">
-        <mass>${m}</mass>
-        <inertia>
-            <ixx>${m*(y*y+z*z)/12}</ixx>
-            <ixy>0</ixy>
-            <ixz>0</ixz>
-            <iyy>${m*(x*x+z*z)/12}</iyy>
-            <iyz>0</iyz>
-            <izz>${m*(x*x+y*y)/12}</izz>
-        </inertia>
-    </xacro_macro_define>
+    <xacro_define_property name="h" value="0.2" />
     <!--rplidar a2-->
     <model name='rplidar_a2'>
@@ -18,5 +7,5 @@
             <inertial>
                 <pose>0 0 0.02 0 0 0</pose>
-                <xacro_macro macro_name="inertia_box" m="0.5" x="${h}" y="${h+0.1}" z="${2*h}"/>
+                <xacro_macro name="inertia_box" m="0.5" x="${h}" y="${h+0.1}" z="${2*h}"/>
             </inertial>
             <collision name="collision">

File: xacro4sdf/common.xacro (robot description, xacro)
@@ -2,5 +2,5 @@
 <sdf version="1.7">
     <!--macro defination:inertia_cylinder-->
-    <xacro_macro_define macro_name="inertia_cylinder" params="m r l">
+    <xacro_define_macro name="inertia_cylinder" params="m r l">
         <mass>${m}</mass>
         <inertia>
@@ -12,7 +12,7 @@
             <izz>${m*r*r/2}</izz>
         </inertia>
-    </xacro_macro_define>
+    </xacro_define_macro>
     <!--macro defination:inertia_box-->
-    <xacro_macro_define macro_name="inertia_box" params="m x y z">
+    <xacro_define_macro name="inertia_box" params="m x y z">
         <mass>${m}</mass>
         <inertia>
@@ -24,7 +24,7 @@
             <izz>${m*(x*x+y*y)/12}</izz>
         </inertia>
-    </xacro_macro_define>
+    </xacro_define_macro>
     <!--macro defination:geometry cylinder-->
-    <xacro_macro_define macro_name="geometry_cylinder" params="r l">
+    <xacro_define_macro name="geometry_cylinder" params="r l">
         <geometry>
             <cylinder>
@@ -33,7 +33,7 @@
             </cylinder>
         </geometry>
-    </xacro_macro_define>
+    </xacro_define_macro>
     <!--macro defination:geometry box-->
-    <xacro_macro_define macro_name="geometry_box" params="x y z">
+    <xacro_define_macro name="geometry_box" params="x y z">
         <geometry>
             <box>
@@ -41,7 +41,7 @@
             </box>
         </geometry>
-    </xacro_macro_define>
+    </xacro_define_macro>
     <!--macro defination:geometry mesh-->
-    <xacro_macro_define macro_name="geometry_mesh" params="filename">
+    <xacro_define_macro name="geometry_mesh" params="filename">
         <geometry>
             <mesh>
@@ -49,7 +49,7 @@
             </mesh>
         </geometry>
-    </xacro_macro_define>
+    </xacro_define_macro>
     <!--macro defination:visual_collision_with_mesh-->
-    <xacro_macro_define macro_name="visual_collision_with_mesh" params="prefix filename">
+    <xacro_define_macro name="visual_collision_with_mesh" params="prefix filename">
         <visual name="${prefix}_visual">
             <geometry>
@@ -66,4 +66,4 @@
             </geometry>
         </collision>
-    </xacro_macro_define>
+    </xacro_define_macro>
 </sdf>

Commit message: update README and test example

File: test/model.sdf.xacro (robot description, xacro)
@@ -10,12 +10,8 @@
             </inertial>
             <collision name="collision">
-                <geometry>
-                    <mesh filename="model://rplidar_a2/meshes/rplidar_a2.dae"/>
-                </geometry>
+                <xacro_macro name="geometry_mesh" uri="model://rplidar_a2/meshes/rplidar_a2.dae"/>
             </collision>
             <visual name="visual">
-                <geometry>
-                    <mesh filename="model://rplidar_a2/meshes/rplidar_a2.dae"/>
-                </geometry>
+                <xacro_macro name="geometry_mesh" uri="model://rplidar_a2/meshes/rplidar_a2.dae"/>
             </visual>
         </link>

Commit message: add support to include xacro definition recursively

File: test/model.sdf.xacro (robot description, xacro)
@@ -1,5 +1,13 @@
 <?xml version="1.0"?>
 <sdf version="1.7">
-    <xacro_define_property name="h" value="0.2" />
+    <xacro_define_property name="rplidar_a2_h" value="0.2" />
+    <xacro_define_macro name = "rplidar_a2_collision_and_visual" params="prefix">
+        <collision name="${prefix}_collision">
+            <xacro_macro name="geometry_mesh" uri="model://rplidar_a2/meshes/rplidar_a2.dae"/>
+        </collision>
+        <visual name="${prefix}_visual">
+            <xacro_macro name="geometry_mesh" uri="model://rplidar_a2/meshes/rplidar_a2.dae"/>
+        </visual>
+    </xacro_define_macro>
     <!--rplidar a2-->
     <model name='rplidar_a2'>
@@ -7,12 +15,7 @@
             <inertial>
                 <pose>0 0 0.02 0 0 0</pose>
-                <xacro_macro name="inertia_box" m="0.5" x="${h}" y="${h+0.1}" z="${2*h}"/>
+                <xacro_macro name="inertia_box" m="0.5" x="${rplidar_a2_h}" y="${rplidar_a2_h+0.1}" z="${2*rplidar_a2_h}"/>
             </inertial>
-            <collision name="collision">
-                <xacro_macro name="geometry_mesh" uri="model://rplidar_a2/meshes/rplidar_a2.dae"/>
-            </collision>
-            <visual name="visual">
-                <xacro_macro name="geometry_mesh" uri="model://rplidar_a2/meshes/rplidar_a2.dae"/>
-            </visual>
+            <xacro_macro name="rplidar_a2_collision_and_visual" prefix="rplidar_a2"/>
         </link>
     </model>
